File: PCB/OE PyBoard.kicad_sch (KiCad schematic)
At the start: 64 parts, among them J1 Conn_01x08, J10 USB4105-GF-A, J11 Micro_SD_Card, J3 Conn_01x08, J4 Conn_01x08, J5 Conn_02x04_Odd_Even, J8 Conn_02x03_Odd_Even, J9 Conn_01x08, U1 STM32F405RGT6, U2 MCP1700T, U4 FXLS8971CFR1, X1 12 MHz, X2 32.768 kHz

Commit message: OE-PyBoard - revisão depois de avaliação Filipe
- nome do projecto/ficheiros alterados para OE-PyBoard
- Colocar OEPS logo para o bottom, e colocar no meio da board
- X1: Mudar a referência para a parte de cima
- udar o diode D1 para 2A & aumentar a secção das linhas VBUS
- alterado o sinal VIN para V+, para ficar coerente com a board original
- passar X2 & C21 & C22 para assembled
- R1=0R passada a solder-jumper
- acrescentadas Labels nos pinos laterais

- gerados production-files
Parts:
- C10: renamed from C11; value 100n -> 100nF
- C15: renamed from C1; value 2u2 -> 2.2uF
- C16: renamed from C2; value 4u7 -> 4.7uF
- C17: value 4.7u -> 4.7uF
- C18: value 100n -> 100nF
- C19: renamed from C21; now fitted; now in the parts list
- C2: renamed from C20; value 100n -> 100nF
- C20: renamed from C22; now fitted; now in the parts list
- C21: renamed from C9; value 100n -> 100nF
- C22: renamed from C6; value 100n -> 100nF
- C3: renamed from C16; value 4.7u -> 4.7uF
- C4: renamed from C15; value 100n -> 100nF
- C5: renamed from C14; value 100n -> 100nF
- C6: renamed from C13; value 100n -> 100nF
- C7: renamed from C12; value 100n -> 100nF
- C8: renamed from C4; value 2u2 -> 2.2uF
- C9: renamed from C5; value 2u2 -> 2.2uF
- D2: renamed from D1; footprint Diode_SMD:D_SOD-123F -> Diode_SMD:D_SOD-128
- J4: renamed from J8; MPN - -> 67996-206HLF; OEPSPN n.a. -> OEPS070015; now in the parts list
- J9: renamed from J5; OEPSPN n.a. -> OEPS00000
- JP2: renamed from R1; footprint Resistor_SMD:R_0402_1005Metric -> Jumper:SolderJumper-2_P1.3mm_Open_RoundedPad1.0x1.5mm; symbol Device:R_Small_US -> Jumper:SolderJumper_2_Open; MPN RC0402JR-070RL -> -; OEPSPN OEPS020001 -> OEPS00000; notes (none) -> n.a.; now fitted
- R10: renamed from R12; MPN CRCW04021M00FKED -> ERJ-2RKF4701X; OEPSPN OEPS020026 -> OEPS020010
- R11: renamed from R13; MPN CRCW04021M00FKED -> ERJ-2RKF4701X; OEPSPN OEPS020026 -> OEPS020010
- R12: renamed from R14; MPN CRCW04021M00FKED -> ERJ-2RKF4701X; OEPSPN OEPS020026 -> OEPS020010
- R13: renamed from R15; MPN CRCW04021M00FKED -> ERJ-2RKF4701X; OEPSPN OEPS020026 -> OEPS020010
- R17: renamed from R16; MPN CRCW04021M00FKED -> ERJ-2RKF4701X; OEPSPN OEPS020026 -> OEPS020010
- R21: MPN CRCW04021M00FKED -> ERJ-2RKF4701X; OEPSPN OEPS020026 -> OEPS020010
- U4: MPN FXLS8971CFR1 -> -; OEPSPN n.a. -> OEPS00000
- X3: renamed from X2; now fitted; now in the parts list
- renumbered C19 to C11, C23 to C12, C7 to C13, C8 to C14, D2 to D3, D3 to D4, D4 to D5, D5 to D6, FB1 to FB2, J11 to J2, J10 to J3, J4 to J5, J9 to J6, J1 to J7, J3 to J8, R10 to R14, R11 to R15, R20 to R16, R6 to R18, R7 to R19, R8 to R20, R9 to R22, R24 to R3, R23 to R4, R4 to R5, R19 to R6, R3 to R7, R22 to R8, R18 to R9, RST1 to RST2, U1 to U2, U2 to U3, USR1 to USR2, X1 to X2
Connections:
- net VIN: no longer C15.1, D2.1 (K), J6.16 (Pin_16), J7.1 (Pin_1), JP2.2, U3.3 (VI)
- new net V+: C15.1, D2.1 (K), J6.16 (Pin_16), J7.1 (Pin_1), JP2.2 (B), U3.3 (VI)
Other:
- note added: "OE Pyboard rev.A"
- note removed: ". 32kHz crystal used 'only' to SD-Card . since SD-card won't be used, does Crystal needs to be assmbled? . is OSC-pins needed to other micro functionalities?"
- note removed: "Test points for JTAG debug available on bottom connector Note: LED resistors may need to be removed for debug (tbd)."
- note removed: "be SURE about FB1 is a ferrite main circuit doesn't let to be sure about"
- moved on the sheet: J9
