File: PCB/OE PyBoard.kicad_sch (KiCad schematic)
At the start: 64 parts, among them J2 Micro_SD_Card, J3 USB4105-GF-A, J4 Conn_02x03_Odd_Even, J5 Conn_01x08, J6 Conn_01x08, J7 Conn_01x08, J8 Conn_01x08, J9 Conn_02x04_Odd_Even, U2 STM32F405RGT6, U3 MCP1700T, U4 FXLS8971CFR1, X2 12 MHz, X3 32.768 kHz

Commit message: sincronia com mudanças q o Filipe fez
Parts:
- J6, J7: MPN SAM1087-16-ND -> CES-116-01-T-S
- R5, R7: value 22R -> 27R
Changed lines of the file:
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@@
 			)
 		)
-		(property "Value" "22R"
+		(property "Value" "27R"
 			(at 89.916 80.01 90)
 			(effects
@@
 			)
 		)
-		(property "MPN" "SAM1087-16-ND"
+		(property "MPN" "CES-116-01-T-S"
 			(at 379.73 198.12 0)
 			(effects
@@
 			)
 		)
-		(property "Value" "22R"
+		(property "Value" "27R"
 			(at 89.662 83.312 90)
 			(effects
@@
 			)
 		)
-		(property "MPN" "SAM1087-16-ND"
+		(property "MPN" "CES-116-01-T-S"
 			(at 328.93 198.12 0)
 			(effects
