File: PCB/OE PyBoard.kicad_pcb (KiCad board)
At the start: 4 copper layers, 33 x 41.9 mm, 57 parts, among them J3 USB4105-GF-A, J4 Conn_02x03_Odd_Even, J6 Conn_01x08, J7 Conn_01x08, U2 STM32F405RGT6, U3 MCP1700T, X2 12 MHz, X3 32.768 kHz

Commit message: sincronia com mudanças q o Filipe fez
Parts:
- R5, R7: value 22R -> 27R
